File: CoilFiringBoard_Hardware/CoilFiringBoard_Hardware.kicad_sch (KiCad schematic)
At the start: 18 parts, among them Q1 Q_NMOS_GDS, Q2 Q_NMOS_GDS

Commit message: bom generated with prices
Parts:
- C1: Price (none) -> 0.46
- D1, D2, D3, D4: Price (none) -> 0.37
- H1, H2: Price (none) -> 2.38
- Q1, Q2: Price (none) -> 18.22
- R1, R2: Price (none) -> 0.33
Changed lines of the file:
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@@
       (effects (font (size 1.27 1.27)) hide)
     )
-    (property "Datasheet" "https://www.digikey.com/en/products/detail/diodes-incorporated/1N5408G-T/128597" (at 153.67 67.31 0)
+    (property "Datasheet" "https://www.mouser.com/ProductDetail/Diodes-Incorporated/1N5408G-T?qs=rGAXPo9uwV2%252BBTeZDYXWZA%3D%3D" (at 153.67 67.31 0)
       (effects (font (size 1.27 1.27)) hide)
     )
@@
       (effects (font (size 1.27 1.27)) hide)
     )
+    (property "Price" "0.37" (at 153.67 67.31 0)
+      (effects (font (size 1.27 1.27)) hide)
+    )
     (pin "1")
     (pin "2")
@@
       (effects (font (size 1.524 1.524)) hide)
     )
+    (property "Price" "" (at 104.14 69.85 0)
+      (effects (font (size 1.27 1.27)) hide)
+    )
     (pin "1")
     (instances
@@
       (effects (font (size 1.27 1.27)) hide)
     )
-    (property "Datasheet" "~" (at 133.35 101.6 0)
+    (property "Datasheet" "https://www.mouser.com/ProductDetail/Panasonic/ERJ-P03F4701V?qs=18kBAoNi3c9lrldXCbY57g%3D%3D" (at 133.35 101.6 0)
+      (effects (font (size 1.27 1.27)) hide)
+    )
+    (property "Price" "0.33" (at 133.35 101.6 0)
       (effects (font (size 1.27 1.27)) hide)
     )
@@
       (effects (font (size 1.27 1.27)) hide)
     )
-    (property "Datasheet" "https://www.digikey.com/en/products/detail/diodes-incorporated/1N5408G-T/128597" (at 161.29 67.31 0)
+    (property "Datasheet" "https://www.mouser.com/ProductDetail/Diodes-Incorporated/1N5408G-T?qs=rGAXPo9uwV2%252BBTeZDYXWZA%3D%3D" (at 161.29 67.31 0)
       (effects (font (size 1.27 1.27)) hide)
     )
@@
       (effects (font (size 1.27 1.27)) hide)
     )
+    (property "Price" "0.37" (at 161.29 67.31 0)
+      (effects (font (size 1.27 1.27)) hide)
+    )
     (pin "1")
     (pin "2")
@@
       (effects (font (size 1.524 1.524)) hide)
     )
+    (property "Price" "" (at 96.52 63.5 0)
+      (effects (font (size 1.27 1.27)) hide)
+    )
     (pin "1")
     (instances
@@
       (effects (font (size 1.27 1.27)) hide)
     )
-    (property "Datasheet" "" (at 180.34 99.06 0)
+    (property "Datasheet" "https://www.mouser.com/ProductDetail/Ohmite/WV-T264-101E?qs=5Eq9T6ZtkovUBRE50m8gYQ%3D%3D" (at 180.34 99.06 0)
+      (effects (font (size 1.27 1.27)) hide)
+    )
+    (property "Price" "2.38" (at 180.34 99.06 0)
       (effects (font (size 1.27 1.27)) hide)
     )
@@
       (effects (font (size 1.27 1.27)) hide)
     )
-    (property "Datasheet" "~" (at 119.38 116.84 0)
+    (property "Datasheet" "~https://www.mouser.com/ProductDetail/KEMET/R60QF14704001K?qs=w%2Fv1CP2dgqrzz3BW9Lijdg%3D%3D" (at 119.38 116.84 0)
+      (effects (font (size 1.27 1.27)) hide)
+    )
+    (property "Price" "0.46" (at 119.38 116.84 0)
       (effects (font (size 1.27 1.27)) hide)
     )
@@
       (effects (font (size 1.27 1.27)) hide)
     )
-    (property "Datasheet" "" (at 193.04 99.06 0)
+    (property "Datasheet" "https://www.mouser.com/ProductDetail/Ohmite/WV-T264-101E?qs=5Eq9T6ZtkovUBRE50m8gYQ%3D%3D" (at 193.04 99.06 0)
+      (effects (font (size 1.27 1.27)) hide)
+    )
+    (property "Price" "2.38" (at 193.04 99.06 0)
       (effects (font (size 1.27 1.27)) hide)
     )
@@
     (property "Datasheet" "" (at 134.62 73.66 0)
       (effects (font (size 1.524 1.524)) hide)
+    )
+    (property "Price" "" (at 134.62 73.66 0)
+      (effects (font (size 1.27 1.27)) hide)
     )
     (pin "1")
@@
       (effects (font (size 1.27 1.27)) hide)
     )
+    (property "Price" "18.22" (at 143.51 83.82 0)
+      (effects (font (size 1.27 1.27)) hide)
+    )
     (pin "1")
     (pin "2")
@@
       (effects (font (size 1.524 1.524)) hide)
     )
+    (property "Price" "" (at 134.62 60.96 0)
+      (effects (font (size 1.27 1.27)) hide)
+    )
     (pin "1")
     (instances
@@
       (effects (font (size 1.27 1.27)) hide)
     )
-    (property "Datasheet" "~" (at 151.13 101.6 0)
+    (property "Datasheet" "https://www.mouser.com/ProductDetail/Panasonic/ERJ-P03F4701V?qs=18kBAoNi3c9lrldXCbY57g%3D%3D" (at 151.13 101.6 0)
+      (effects (font (size 1.27 1.27)) hide)
+    )
+    (property "Price" "0.33" (at 151.13 101.6 0)
       (effects (font (size 1.27 1.27)) hide)
     )
@@
       (effects (font (size 1.27 1.27)) hide)
     )
-    (property "Datasheet" "https://www.digikey.com/en/products/detail/diodes-incorporated/1N5408G-T/128597" (at 168.91 67.31 0)
+    (property "Datasheet" "https://www.mouser.com/ProductDetail/Diodes-Incorporated/1N5408G-T?qs=rGAXPo9uwV2%252BBTeZDYXWZA%3D%3D" (at 168.91 67.31 0)
       (effects (font (size 1.27 1.27)) hide)
     )
@@
     )
     (property "Sim.Pins" "1=K 2=A" (at 168.91 67.31 0)
+      (effects (font (size 1.27 1.27)) hide)
+    )
+    (property "Price" "0.37" (at 168.91 67.31 0)
       (effects (font (size 1.27 1.27)) hide)
     )
@@
       (effects (font (size 1.27 1.27)) hide)
     )
+    (property "Price" "18.22" (at 161.29 83.82 0)
+      (effects (font (size 1.27 1.27)) hide)
+    )
     (pin "1")
     (pin "2")
@@
     (property "Datasheet" "" (at 104.14 63.5 0)
       (effects (font (size 1.524 1.524)) hide)
+    )
+    (property "Price" "" (at 104.14 63.5 0)
+      (effects (font (size 1.27 1.27)) hide)
     )
     (pin "1")
@@
       (effects (font (size 1.524 1.524)) hide)
     )
+    (property "Price" "" (at 105.41 95.25 0)
+      (effects (font (size 1.27 1.27)) hide)
+    )
     (pin "1")
     (pin "2")
@@
       (effects (font (size 1.27 1.27)) hide)
     )
-    (property "Datasheet" "https://www.digikey.com/en/products/detail/diodes-incorporated/1N5408G-T/128597" (at 146.05 67.31 0)
+    (property "Datasheet" "https://www.mouser.com/ProductDetail/Diodes-Incorporated/1N5408G-T?qs=rGAXPo9uwV2%252BBTeZDYXWZA%3D%3D" (at 146.05 67.31 0)
       (effects (font (size 1.27 1.27)) hide)
     )
@@
       (effects (font (size 1.27 1.27)) hide)
     )
+    (property "Price" "0.37" (at 146.05 67.31 0)
+      (effects (font (size 1.27 1.27)) hide)
+    )
     (pin "1")
     (pin "2")
@@
       (effects (font (size 1.524 1.524)) hide)
     )
-    (pin "1")
+    (property "Price" "" (at 96.52 69.85 0)
+      (effects (font (size 1.27 1.27)) hide)
+    )
+    (pin "1")
